Commit message: added inertia elements to support use in gazebo

File: abb_irb4600_support/urdf/irb4600_40_255_macro.xacro (robot description, xacro)
@@ -5,4 +5,8 @@
     <!-- link list -->
     <link name="${prefix}base_link">
+      <inertial>
+        <mass value="0.1" />
+        <inertia ixx="0.03" iyy="0.03" izz="0.03" ixy="0.0" ixz="0.0" iyz="0.0" />
+      </inertial>
       <collision name="collision">
         <geometry>
@@ -22,4 +26,8 @@
     </link>
     <link name="${prefix}link_1">
+      <inertial>
+        <mass value="0.1" />
+        <inertia ixx="0.03" iyy="0.03" izz="0.03" ixy="0.0" ixz="0.0" iyz="0.0" />
+      </inertial>
       <collision name="collision">
         <geometry>
@@ -37,4 +45,8 @@
     </link>
     <link name="${prefix}link_2">
+      <inertial>
+        <mass value="0.1" />
+        <inertia ixx="0.03" iyy="0.03" izz="0.03" ixy="0.0" ixz="0.0" iyz="0.0" />
+      </inertial>
       <collision name="collision">
         <geometry>
@@ -52,4 +64,8 @@
     </link>
     <link name="${prefix}link_3">
+      <inertial>
+        <mass value="0.1" />
+        <inertia ixx="0.03" iyy="0.03" izz="0.03" ixy="0.0" ixz="0.0" iyz="0.0" />
+      </inertial>
       <collision name="collision">
         <geometry>
@@ -67,4 +83,8 @@
     </link>
     <link name="${prefix}link_4">
+      <inertial>
+        <mass value="0.1" />
+        <inertia ixx="0.03" iyy="0.03" izz="0.03" ixy="0.0" ixz="0.0" iyz="0.0" />
+      </inertial>
       <collision name="collision">
         <geometry>
@@ -82,4 +102,8 @@
     </link>
     <link name="${prefix}link_5">
+      <inertial>
+        <mass value="0.1" />
+        <inertia ixx="0.03" iyy="0.03" izz="0.03" ixy="0.0" ixz="0.0" iyz="0.0" />
+      </inertial>
       <collision name="collision">
         <geometry>
@@ -97,4 +121,8 @@
     </link>
     <link name="${prefix}link_6">
+      <inertial>
+        <mass value="0.1" />
+        <inertia ixx="0.03" iyy="0.03" izz="0.03" ixy="0.0" ixz="0.0" iyz="0.0" />
+      </inertial>
       <collision name="collision">
         <geometry>

Commit message: chnaged location of joint_3 to be correct.

File: abb_irb4600_support/urdf/irb4600_40_255_macro.xacro (robot description, xacro)
@@ -13,14 +13,11 @@
           <mesh filename="package://abb_irb4600_support/meshes/irb4600_common/collision/base_link.stl"/>
         </geometry>
-        <xacro:material_abb_white/>
+        <xacro:material_abb_olive_green/>
       </collision>
-      <visual name="visual">
+      <visual>
         <geometry>
           <mesh filename="package://abb_irb4600_support/meshes/irb4600_common/visual/base_link.stl"/>
         </geometry>
-        <xacro:material_abb_white/>
-        <material name="yellow">
-          <color rgba="1 1 0 1"/>
-        </material>
+        <xacro:material_abb_olive_green/>>
       </visual>
     </link>
@@ -34,11 +31,11 @@
           <mesh filename="package://abb_irb4600_support/meshes/irb4600_common/collision/link_1.stl"/>
         </geometry>
-        <xacro:material_abb_white/>
+        <xacro:material_abb_olive_green/>
       </collision>
-      <visual name="visual">
+      <visual>
         <geometry>
           <mesh filename="package://abb_irb4600_support/meshes/irb4600_common/visual/link_1.stl"/>
         </geometry>
-        <xacro:material_abb_white/>
+        <xacro:material_abb_olive_green/>
         <material name="yellow"/>
       </visual>
@@ -53,11 +50,11 @@
           <mesh filename="package://abb_irb4600_support/meshes/irb4600_40_255/collision/link_2.stl"/>
         </geometry>
-        <xacro:material_abb_white/>
+        <xacro:material_abb_olive_green/>
       </collision>
-      <visual name="visual">
+      <visual>
         <geometry>
           <mesh filename="package://abb_irb4600_support/meshes/irb4600_40_255/visual/link_2.stl"/>
         </geometry>
-        <xacro:material_abb_white/>
+        <xacro:material_abb_olive_green/>
         <material name="yellow"/>
       </visual>
@@ -72,11 +69,11 @@
           <mesh filename="package://abb_irb4600_support/meshes/irb4600_40_255/collision/link_3.stl"/>
         </geometry>
-        <xacro:material_abb_white/>
+        <xacro:material_abb_olive_green/>
       </collision>
-      <visual name="visual">
+      <visual>
         <geometry>
           <mesh filename="package://abb_irb4600_support/meshes/irb4600_40_255/visual/link_3.stl"/>
         </geometry>
-        <xacro:material_abb_white/>
+        <xacro:material_abb_olive_green/>
         <material name="yellow"/>
       </visual>
@@ -91,11 +88,11 @@
           <mesh filename="package://abb_irb4600_support/meshes/irb4600_40_255/collision/link_4.stl"/>
         </geometry>
-        <xacro:material_abb_white/>
+        <xacro:material_abb_olive_green/>
       </collision>
-      <visual name="visual">
+      <visual>
         <geometry>
           <mesh filename="package://abb_irb4600_support/meshes/irb4600_40_255/visual/link_4.stl"/>
         </geometry>
-        <xacro:material_abb_white/>
+        <xacro:material_abb_olive_green/>
         <material name="yellow"/>
       </visual>
@@ -110,12 +107,11 @@
           <mesh filename="package://abb_irb4600_support/meshes/irb4600_40_255/collision/link_5.stl"/>
         </geometry>
-        <xacro:material_abb_white/>
+        <xacro:material_abb_olive_green/>
       </collision>
-      <visual name="visual">
+      <visual>
         <geometry>
           <mesh filename="package://abb_irb4600_support/meshes/irb4600_40_255/visual/link_5.stl"/>
         </geometry>
-        <xacro:material_abb_white/>
-        <material name="yellow"/>
+        <xacro:material_abb_olive_green/>
       </visual>
     </link>
@@ -129,11 +125,11 @@
           <mesh filename="package://abb_irb4600_support/meshes/irb4600_40_255/collision/link_6.stl"/>
         </geometry>
-        <xacro:material_abb_white/>
+        <xacro:material_abb_olive_green/>
       </collision>
-      <visual name="visual">
+      <visual>
         <geometry>
           <mesh filename="package://abb_irb4600_support/meshes/irb4600_40_255/visual/link_6.stl"/>
         </geometry>
-        <xacro:material_abb_white/>
+        <xacro:material_abb_olive_green/>
         <material name="yellow"/>
       </visual>
@@ -157,5 +153,5 @@
     </joint>
     <joint type="revolute" name="${prefix}joint_3">
-      <origin xyz="0 0 0.9" rpy="0 0 0"/>
+      <origin xyz="0 0 1.095" rpy="0 0 0"/>
       <axis xyz="0 1 0"/>
       <parent link="${prefix}link_2"/>
